Commit message: add inertia shortcuts

File: urdf/common_properties.urdf.xacro (robot description, xacro)
@@ -2,4 +2,29 @@
 <!-- Various useful macros -->
 <robot name="xacro_properties" xmlns:xacro="http://ros.org/wiki/xacro">
+    <xacro:macro name="cuboid_inertia" params="mass x y z">
+        <inertial>
+            <mass value="${mass}" />
+            <inertia ixx="${(1/12) * mass * (y*y + z*z)}" ixy="0.0" ixz="0.0"
+                iyy="${(1/12) * mass * (x*x + z*z)}" iyz="0.0"
+                izz="${(1/12) * mass * (x*x + y*y)}" />
+        </inertial>
+    </xacro:macro>
+    <xacro:macro name="sphere_inertia" params="mass radius">
+        <inertial>
+            <mass value="${mass}" />
+            <inertia ixx="${(2/5) * mass * radius * radius}" ixy="0.0" ixz="0.0"
+                iyy="${(2/5) * mass * radius * radius}" iyz="0.0"
+                izz="${(2/5) * mass * radius * radius}" />
+        </inertial>
+    </xacro:macro>
+    <xacro:macro name="cylinder_inertia" params="mass radius length">
+        <inertial>
+            <mass value="${mass}" />
+            <inertia ixx="${(1/12) * mass * (3*radius*radius + length*length)}" ixy="0.0" ixz="0.0"
+                iyy="${(1/12) * mass * (3*radius*radius + length*length)}" iyz="0.0"
+                izz="${(1/2) * mass * (radius*radius)}" />
+        </inertial>
+    </xacro:macro>
+    <!-- others -->
     <xacro:macro name="inertial_cuboid_with_pose" params="mass x y z *origin">
         <inertial>
