Commit message: update launch files and urdf

File: urdf/robot.urdf (robot description, URDF)
Before this commit: robot robot, 1 links, 0 joints
Links:
- added link base_link
- added link front_left_wheel, mass 11.0; collision sphere radius=0.25; visual cylinder length=0.15 radius=0.25
- added link front_left_wheel_steering_link, mass 1.0
- added link front_right_wheel, mass 11.0; collision sphere radius=0.25; visual cylinder length=0.15 radius=0.25
- added link front_right_wheel_steering_link, mass 1.0
- added link rear_left_wheel, mass 11.0; collision sphere radius=0.25; visual cylinder length=0.15 radius=0.25
- added link rear_right_wheel, mass 11.0; collision sphere radius=0.25; visual cylinder length=0.15 radius=0.25
- link link_chassis: mass 10 -> 500.0; geometry collision box size=1.0 1.0 0.5; visual mesh filename=package://gazebo_project/meshes/smart_car.obj scale=0.012 0.012 0.013
Joints:
- added joint front_left_wheel_rotating_joint: type revolute, parent front_left_wheel_steering_link, child front_left_wheel, origin xyz=0 0 0 rpy=0 0 0, axis 0 0 1, limit lower=-1.79769e+308 upper=1.79769e+308 effort=100000 velocity=1000
- added joint front_left_wheel_steering_joint: type revolute, parent link_chassis, child front_left_wheel_steering_link, origin xyz=0.9 0.64 0.25 rpy=-1.56 0 0, axis 0 -1 0, limit lower=-0.8727 upper=0.8727 effort=100000 velocity=1000
- added joint front_right_wheel_rotating_joint: type revolute, parent front_right_wheel_steering_link, child front_right_wheel, origin xyz=0 0 0 rpy=0 0 0, axis 0 0 1, limit lower=-1.79769e+308 upper=1.79769e+308 effort=100000 velocity=1000
- added joint front_right_wheel_steering_joint: type revolute, parent link_chassis, child front_right_wheel_steering_link, origin xyz=0.9 -0.64 0.25 rpy=-1.56 0 0, axis 0 -1 0, limit lower=-0.8727 upper=0.8727 effort=100000 velocity=1000
- added joint joint_base_link_chassis: type fixed, parent base_link, child link_chassis, origin xyz=0 0 0 rpy=0 0 0
- added joint rear_left_wheel_joint: type revolute, parent link_chassis, child rear_left_wheel, origin xyz=-0.9 0.64 0.25 rpy=1.56 0 0, axis 0 0 1, limit lower=-1.79769e+308 upper=1.79769e+308 effort=100000 velocity=1000
- added joint rear_right_wheel_joint: type revolute, parent link_chassis, child rear_right_wheel, origin xyz=-0.9 -0.64 0.25 rpy=1.56 0 0, axis 0 0 1, limit lower=-1.79769e+308 upper=1.79769e+308 effort=100000 velocity=1000

Commit message: fix inertias

File: urdf/robot.urdf (robot description, URDF)
Before this commit: robot robot, 8 links, 7 joints
Links:
- link front_left_wheel: mass 11.0 -> None
- link front_left_wheel_steering_link: mass 1.0 -> None
- link front_right_wheel: mass 11.0 -> None
- link front_right_wheel_steering_link: mass 1.0 -> None
- link link_chassis: mass 500.0 -> None; geometry collision box size=2.4 1.0 1.0; visual mesh filename=package://gazebo_project/meshes/smart_car.obj scale=0.012 0.012 0.013
- link rear_left_wheel: mass 11.0 -> None
- link rear_right_wheel: mass 11.0 -> None

Commit message: add hw

File: urdf/robot.urdf (robot description, URDF)
Before this commit: robot robot, 8 links, 7 joints
Links:
- removed link front_left_wheel
- removed link front_left_wheel_steering_link
- removed link front_right_wheel
- removed link front_right_wheel_steering_link
- removed link link_chassis
- removed link rear_left_wheel
- removed link rear_right_wheel
Joints:
- removed joint front_left_wheel_rotating_joint
- removed joint front_left_wheel_steering_joint
- removed joint front_right_wheel_rotating_joint
- removed joint front_right_wheel_steering_joint
- removed joint joint_base_link_chassis
- removed joint rear_left_wheel_joint
- removed joint rear_right_wheel_joint
