Commit message: change camera position

File: urdf/oakd.urdf.xacro (robot description, xacro)
@@ -104,8 +104,8 @@
             <sensor name="rgbd_camera" type="rgbd_camera">
                 <camera>
-                    <horizontal_fov>1.25</horizontal_fov>
+                    <horizontal_fov>2.2</horizontal_fov>
                     <image>
-                        <width>320</width>
-                        <height>240</height>
+                        <width>1080</width>
+                        <height>720</height>
                     </image>
                     <clip>
@@ -116,5 +116,5 @@
                 </camera>
                 <always_on>1</always_on>
-                <update_rate>30</update_rate>
+                <update_rate>6</update_rate>
                 <visualize>true</visualize>
             </sensor>

File: urdf/robot.urdf (robot description, URDF)
Before this commit: robot robot, 1 links, 0 joints
Links:
- added link front_left_wheel; collision sphere radius=0.25; visual cylinder length=0.15 radius=0.25
- added link front_left_wheel_steering_link
- added link front_right_wheel; collision sphere radius=0.25; visual cylinder length=0.15 radius=0.25
- added link front_right_wheel_steering_link
- added link link_chassis; collision box size=2.4 1.0 1.0; visual mesh filename=package://gazebo_project/meshes/smart_car.obj scale=0.012 0.012 0.013
- added link rear_left_wheel; collision sphere radius=0.25; visual cylinder length=0.15 radius=0.25
- added link rear_right_wheel; collision sphere radius=0.25; visual cylinder length=0.15 radius=0.25
Joints:
- added joint front_left_wheel_rotating_joint: type revolute, parent front_left_wheel_steering_link, child front_left_wheel, origin xyz=0 0 0 rpy=0 0 0, axis 0 0 1, limit lower=-1.79769e+308 upper=1.79769e+308 effort=100 velocity=20
- added joint front_left_wheel_steering_joint: type revolute, parent link_chassis, child front_left_wheel_steering_link, origin xyz=0.9 0.64 0.25 rpy=-1.56 0 0, axis 0 -1 0, limit lower=-0.8727 upper=0.8727 effort=100000 velocity=1000
- added joint front_right_wheel_rotating_joint: type revolute, parent front_right_wheel_steering_link, child front_right_wheel, origin xyz=0 0 0 rpy=0 0 0, axis 0 0 1, limit lower=-1.79769e+308 upper=1.79769e+308 effort=100 velocity=20
- added joint front_right_wheel_steering_joint: type revolute, parent link_chassis, child front_right_wheel_steering_link, origin xyz=0.9 -0.64 0.25 rpy=-1.56 0 0, axis 0 -1 0, limit lower=-0.8727 upper=0.8727 effort=100000 velocity=1000
- added joint joint_base_link_chassis: type fixed, parent base_link, child link_chassis, origin xyz=0 0 0 rpy=0 0 0
- added joint rear_left_wheel_joint: type revolute, parent link_chassis, child rear_left_wheel, origin xyz=-0.9 0.64 0.25 rpy=1.56 0 0, axis 0 0 1, limit lower=-1.79769e+308 upper=1.79769e+308 effort=100000 velocity=1000
- added joint rear_right_wheel_joint: type revolute, parent link_chassis, child rear_right_wheel, origin xyz=-0.9 -0.64 0.25 rpy=1.56 0 0, axis 0 0 1, limit lower=-1.79769e+308 upper=1.79769e+308 effort=100000 velocity=1000
